Commit message: Updated the urdf to match the current build of the real robot

File: src/mws_robot/description/gazebo_control.xacro (robot description, xacro)
@@ -6,8 +6,8 @@
             <left_joint>left_wheel_joint</left_joint>
             <right_joint>right_wheel_joint</right_joint>
-            <wheel_separation>0.46</wheel_separation>
-            <wheel_diameter>0.245</wheel_diameter>
+            <wheel_separation>0.49</wheel_separation>
+            <wheel_diameter>0.0735</wheel_diameter>
             <!-- Limits -->
-            <max_wheel_torque>200</max_wheel_torque>
+            <max_wheel_torque>7</max_wheel_torque>
             <max_wheel_acceleration>10.0</max_wheel_acceleration>
             <!-- Output -->

File: src/mws_robot/description/lidar.xacro (robot description, xacro)
@@ -2,5 +2,5 @@
 <robot xmlns:xacro="http://www.ros.org/wiki/xacro" >
     <xacro:property name="laser_frame_offset_x" value="0.36"/>  <!-- Length and offset is specified in Meters -->
-    <xacro:property name="laser_frame_offset_z" value="1.24"/>
+    <xacro:property name="laser_frame_offset_z" value="1.253"/>
     <xacro:property name="lidar_radius" value="0.05"/>
     <xacro:property name="lidar_length" value="0.04"/>

File: src/mws_robot/description/mws_robot_core.xacro (robot description, xacro)
@@ -4,13 +4,13 @@
     <xacro:property name="chassis_width" value="0.71"/>
     <xacro:property name="chassis_height" value="0.955"/>
-    <xacro:property name="chassis_offset_z" value="0.04"/>
-    <xacro:property name="chassis_offset_x" value="0.22"/>
-    <xacro:property name="chassis_mass" value="25.0"/>  <!-- Mass is specified in Kilograms -->
-    <xacro:property name="wheel_radius" value="0.1225"/>
-    <xacro:property name="wheel_thickness" value="0.05"/>
-    <xacro:property name="wheel_mass" value="3"/>
+    <xacro:property name="chassis_offset_z" value="0.105"/>
+    <xacro:property name="chassis_offset_x" value="0.205"/>
+    <xacro:property name="chassis_mass" value="30.0"/>  <!-- Mass is specified in Kilograms -->
+    <xacro:property name="wheel_radius" value="0.0735"/>
+    <xacro:property name="wheel_thickness" value="0.03"/>
+    <xacro:property name="wheel_mass" value="1.5"/>
     <xacro:property name="wheel_offset_x" value="0.226"/>
-    <xacro:property name="wheel_offset_y" value="0.23"/>
-    <xacro:property name="wheel_offset_z" value="0.1225"/>
+    <xacro:property name="wheel_offset_y" value="0.245"/>
+    <xacro:property name="wheel_offset_z" value="${wheel_radius}"/>
     <xacro:property name="caster_wheel_radius" value="${chassis_offset_z / 2}"/>
     <xacro:property name="caster_wheel_mass" value="1"/>
